File: pcb/camera_link.kicad_pcb (KiCad board)
At the start: 2 copper layers, 159.3 x 14.5 mm, 12 parts, among them J1 RJ45_pyControl, J2 Screw_Terminal_01x08

Commit message: pcbv1.2
Parts:
- removed R2: R_US, Resistor_THT:R_Axial_DIN0204_L3.6mm_D1.6mm_P7.62mm_Horizontal
- added D10: LED, LED_SMD:LED_1206_3216Metric, B.Cu at (157.9, 113.0)
- added D11: LED, LED_SMD:LED_1206_3216Metric, B.Cu at (175.9, 118.0)
- added D12: LED, LED_SMD:LED_1206_3216Metric, B.Cu at (157.9, 123.0)
- added D13: LED, LED_SMD:LED_1206_3216Metric, B.Cu at (139.9, 108.0)
- added D14: LED, LED_SMD:LED_1206_3216Metric, B.Cu at (121.9, 113.0)
- added D15: LED, LED_SMD:LED_1206_3216Metric, B.Cu at (139.9, 118.0)
- added D16: LED, LED_SMD:LED_1206_3216Metric, B.Cu at (121.9, 123.0)
- added D17: LED, LED_SMD:LED_1206_3216Metric, B.Cu at (103.9, 108.0)
- added D18: LED, LED_SMD:LED_1206_3216Metric, B.Cu at (85.9, 113.0)
- added D19: LED, LED_SMD:LED_1206_3216Metric, B.Cu at (103.9, 118.0)
- added D20: LED, LED_SMD:LED_1206_3216Metric, B.Cu at (85.9, 123.0)
- added D21: LED, LED_SMD:LED_1206_3216Metric, B.Cu at (67.9, 108.0)
- added D22: LED, LED_SMD:LED_1206_3216Metric, B.Cu at (49.9, 113.0)
- added D23: LED, LED_SMD:LED_1206_3216Metric, B.Cu at (67.9, 118.0)
- added D24: LED, LED_SMD:LED_1206_3216Metric, B.Cu at (49.9, 123.0)
- added D7: LED, LED_SMD:LED_1206_3216Metric, B.Cu at (211.9, 118.0)
- added D8: LED, LED_SMD:LED_1206_3216Metric, B.Cu at (193.9, 123.0)
- added D9: LED, LED_SMD:LED_1206_3216Metric, B.Cu at (175.9, 108.0)
- J1: footprint asl_footprints:RJ45_THP_Vertical -> asl_footprints:RJ45_SMD
- R1: value R_US -> 9Ω; footprint Resistor_THT:R_Axial_DIN0204_L3.6mm_D1.6mm_P7.62mm_Horizontal -> Resistor_SMD:R_1206_3216Metric_Pad1.30x1.75mm_HandSolder; moved to B.Cu
- moved D1 172.0 mm to (247.9, 108.0), turned to 0 degrees
- moved D4 123.3 mm to (229.9, 123.0), turned to 0 degrees
- moved D2 92.9 mm to (229.9, 112.9), turned to 0 degrees
- moved R1 77.0 mm to (50.8, 108.0), turned to 90 degrees
- moved D3 49.8 mm to (247.9, 118.0), turned to 0 degrees
- moved D5 45.3 mm to (211.9, 108.0), turned to 0 degrees
- moved D6 35.0 mm to (193.9, 113.0), turned to 0 degrees
- moved H2 19.4 mm to (59.7, 115.6)
- moved H1 14.4 mm to (240.0, 115.6)
- moved J1 4.57 mm to (91.9, 104.1)
- moved J2 4.16 mm to (150.3, 112.3), turned to 180 degrees
Connections:
- net Net-(J1-Pad2) renamed /GND
- D1 pad 2: /5VDC -> Net-(D1-Pad2)
- D2 pad 2: /5VDC -> Net-(D1-Pad2)
- D3 pad 2: /5VDC -> Net-(D1-Pad2)
- D4 pad 1: Net-(D4-Pad1) -> Net-(D1-Pad1)
- D4 pad 2: /5VDC -> Net-(D1-Pad2)
- D5 pad 1: Net-(D4-Pad1) -> Net-(D10-Pad2)
- D5 pad 2: /5VDC -> Net-(D1-Pad1)
- D6 pad 1: Net-(D4-Pad1) -> Net-(D10-Pad2)
- D6 pad 2: /5VDC -> Net-(D1-Pad1)
- J1 pad 6: /5VDC -> Net-(J1-Pad6)
- J1 pad 8: Net-(J1-Pad8) -> Net-(D1-Pad2)
- J2 pad 6: /5VDC -> Net-(J1-Pad6)
- J2 pad 8: Net-(J1-Pad8) -> Net-(D1-Pad2)
- R1 pad 1: Net-(J1-Pad7) -> Net-(D21-Pad1)
- R1 pad 2: Net-(D1-Pad1) -> Net-(J1-Pad7)
Routing:
- net Net-(D1-Pad2): track 0.00 -> 202.8 mm, vias 0 -> 1
- net Net-(D4-Pad1): track 133.7 -> 0.00 mm, vias 2 -> 0
- net Net-(D10-Pad1): track 0.00 -> 97.8 mm
- net Net-(D13-Pad1): track 0.00 -> 97.4 mm
- net Net-(D10-Pad2): track 0.00 -> 97.4 mm
- net Net-(D17-Pad1): track 0.00 -> 97.4 mm
- net Net-(J1-Pad8): track 74.4 -> 0.00 mm
- net Net-(J1-Pad6): track 0.00 -> 70.2 mm
- net Net-(D1-Pad1): track 147.5 -> 97.4 mm, vias 4 -> 0
- net Net-(J1-Pad7): track 69.6 -> 115.6 mm
- net Net-(D21-Pad1): track 0.00 -> 40.8 mm
- net Net-(J1-Pad3): track 94.8 -> 61.6 mm
- net /5VDC: track 19.6 -> 0.00 mm, vias 4 -> 0
- net Net-(J1-Pad1): track 47.8 -> 55.9 mm
- net /GND: track 52.0 -> 59.4 mm
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- removed copper zone on B.Cu, net /5VDC
- removed copper zone on F.Cu, net /5VDC
Other:
- board size 159.3 x 14.5 mm -> 203.8 x 22.2 mm
- board text added: "Camera Link v1.2"
- board text added: "DB"
- board text removed: "Camera Link v1.1"

Commit message: pcb v1.3
Parts:
- removed D10, D11, D12, D13, D14, D15, D16, D17, D18, D19, D20, D21, D22, D23, D24, D4, D5, D6, D7, D8, D9: LED, LED_SMD:LED_1206_3216Metric
- added GND_TEST1: TestPoint, Connector_Pin:Pin_D1.0mm_L10.0mm, F.Cu at (192.5, 115.8)
- added GRAB1: TestPoint, Connector_Pin:Pin_D1.0mm_L10.0mm, F.Cu at (142.2, 106.7)
- added J3: Conn_01x09_Female, asl_footprints:JST_NSH_1x09_VERTICAL, F.Cu at (132.6, 114.8)
- added Q1: 2N2219, Package_TO_SOT_SMD:SOT-23-6, F.Cu at (97.8, 122.9)
- added R2: 100, Resistor_SMD:R_0805_2012Metric, F.Cu at (106.7, 115.8)
- added R3: MP915-4.00-1%, asl_footprints:Resistor_power_MP900, F.Cu at (105.4, 123.2)
- added RV1: 3386P-1-504TLF, Potentiometer_THT:Potentiometer_Bourns_3386P_Vertical, F.Cu at (89.5, 117.5)
- added SYNC1: TestPoint, Connector_Pin:Pin_D1.0mm_L10.0mm, F.Cu at (134.6, 122.9)
- added TP1: TestPoint, Connector_Pin:Pin_D1.0mm_L10.0mm, F.Cu at (87.0, 109.0)
- added TP2: TestPoint, Connector_Pin:Pin_D1.0mm_L10.0mm, F.Cu at (87.0, 113.0)
- added U1: LM741, Package_DIP:DIP-8_W7.62mm, F.Cu at (95.8, 109.7)
- D1, D2, D3: value LED -> LST1-01F09-IR01-00; footprint LED_SMD:LED_1206_3216Metric -> asl_footprints:LED_starboard; moved to F.Cu
- H1: renamed from H2; value Threaded_Standoff -> 24882
- H2: renamed from H1; value Threaded_Standoff -> 24882
- J1: value RJ45_pyControl -> 54602-908LF; footprint asl_footprints:RJ45_SMD -> asl_footprints:RJ45_THP
- J2: value Screw_Terminal_01x08 -> Conn_01x09_Female; footprint Connector_PinHeader_1.27mm:PinHeader_1x08_P1.27mm_Vertical -> asl_footprints:JST_NSH_1x09_VERTICAL
- R1: value 9Ω -> 5K; footprint Resistor_SMD:R_1206_3216Metric_Pad1.30x1.75mm_HandSolder -> Resistor_SMD:R_0805_2012Metric; moved to F.Cu
- moved D3 174.9 mm to (73.0, 115.6), turned to 180 degrees
- moved D2 79.8 mm to (150.2, 115.6)
- moved R1 41.2 mm to (91.9, 109.0), turned to -90 degrees
- moved J1 27.7 mm to (118.6, 111.8)
- moved D1 21.9 mm to (227.3, 115.3), turned to 180 degrees
- moved J2 16.0 mm to (166.1, 114.8), turned to 90 degrees
Connections:
- D1 pad 1: Net-(D1-Pad1) -> Net-(D1-K)
- D1 pad 2: Net-(D1-Pad2) -> Net-(D1-A)
- D2 pad 1: Net-(D1-Pad1) -> Net-(D2-K)
- D2 pad 2: Net-(D1-Pad2) -> Net-(D1-K)
- D3 pad 1: Net-(D1-Pad1) -> Net-(D3-K)
- D3 pad 2: Net-(D1-Pad2) -> Net-(D2-K)
- J1 pad 1: Net-(J1-Pad1) -> /GRAB
- J1 pad 2: /GND -> GND
- J1 pad 3: Net-(J1-Pad3) -> unconnected-(J1-POW-A)
- J1 pad 4: Net-(J1-Pad4) -> /SYNC
- J1 pad 5: Net-(J1-Pad5) -> unconnected-(J1-SPECIAL)
- J1 pad 6: Net-(J1-Pad6) -> Net-(J1-5V)
- J1 pad 7: Net-(J1-Pad7) -> /POW_B
- J1 pad 8: Net-(D1-Pad2) -> Net-(D1-A)
- J2 pad 1: Net-(J1-Pad1) -> /SYNC
- J2 pad 2: /GND -> unconnected-(J2-Pin_2)
- J2 pad 3: Net-(J1-Pad3) -> GND
- J2 pad 4: Net-(J1-Pad4) -> GND
- J2 pad 5: Net-(J1-Pad5) -> unconnected-(J2-Pin_5)
- J2 pad 6: Net-(J1-Pad6) -> /GRAB
- J2 pad 7: Net-(J1-Pad7) -> unconnected-(J2-Pin_7)
- J2 pad 8: Net-(D1-Pad2) -> unconnected-(J2-Pin_8)
- R1 pad 1: Net-(D21-Pad1) -> Net-(J1-5V)
- R1 pad 2: Net-(J1-Pad7) -> Net-(R1-Pad2)
Routing:
- net Net-(D1-Pad2): track 202.8 -> 0.00 mm, vias 1 -> 0
- net Net-(D1-A): track 0.00 -> 130.1 mm
- net Net-(J1-Pad7): track 115.6 -> 0.00 mm, vias 1 -> 0
- net Net-(D2-K): track 0.00 -> 102.4 mm
- net Net-(D10-Pad1): track 97.8 -> 0.00 mm
- net Net-(D1-K): track 0.00 -> 97.5 mm
- net Net-(D1-Pad1): track 97.4 -> 0.00 mm
- net Net-(D13-Pad1): track 97.4 -> 0.00 mm
- net Net-(D10-Pad2): track 97.4 -> 0.00 mm
- net Net-(D17-Pad1): track 97.4 -> 0.00 mm
- net Net-(J1-Pad6): track 70.2 -> 0.00 mm
- net Net-(J1-Pad5): track 68.2 -> 0.00 mm
- net Net-(J1-Pad4): track 63.9 -> 0.00 mm
- net Net-(J1-Pad3): track 61.6 -> 0.00 mm
- net /GND: track 59.4 -> 0.00 mm
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- added copper zone on B.Cu, net GND
- added copper zone on F.Cu, net GND
Other:
- board text added: "Camera Link v1.3"
- board text removed: "Camera Link v1.2"
- board text removed: "DA"
- board text removed: "DB"
- board text removed: "GND"

Commit message: pcb v1.5
Parts:
- removed J3: Conn_01x09_Female, asl_footprints:JST_NSH_1x09_VERTICAL
- removed Q1: 2N2219, Package_TO_SOT_SMD:SOT-23-6
- removed the R1 at (91.9, 109.0)
- removed R3: MP915-4.00-1%, asl_footprints:Resistor_power_MP900
- removed RV1: 3386P-1-504TLF, Potentiometer_THT:Potentiometer_Bourns_3386P_Vertical
- removed TP1, TP2: TestPoint, Connector_Pin:Pin_D1.0mm_L10.0mm
- added D1: D, Diode_SMD:D_SMB, F.Cu at (96.5, 111.0)
- added L1: L, Inductor_THT:L_Axial_L14.5mm_D5.8mm_P7.62mm_Vertical_Fastron_HBCC, F.Cu at (88.4, 118.5)
- added R2: R_US, Resistor_SMD:R_0805_2012Metric, F.Cu at (113.8, 123.4)
- J1: value 54602-908LF -> E5J88-00LJG2-L; footprint asl_footprints:RJ45_THP -> asl_footprints:RJ45_THP_tab_on_top
- R1: renamed from R2; value 100 -> R_US; footprint Resistor_SMD:R_0805_2012Metric -> Resistor_THT:R_Axial_DIN0614_L14.3mm_D5.7mm_P7.62mm_Vertical
- U1: value LM741 -> AL8861; footprint Package_DIP:DIP-8_W7.62mm -> Package_TO_SOT_SMD:SOT-89-5
- moved SYNC1 43.3 mm to (177.8, 119.1)
- moved GRAB1 36.7 mm to (177.8, 115.8)
- moved GND1 10.3 mm to (182.4, 117.5)
- moved U1 9.42 mm to (96.5, 119.1)
- moved R1 3.79 mm to (104.9, 112.5)
- moved J1 2.54 mm to (118.6, 109.2)
- moved J2 2.41 mm to (168.4, 115.6)
- turned D3 to 180 degrees
- renumbered D1 to D2, D2 to D3, D3 to D4, GND_TEST1 to GND1, H2 to H1, H1 to H2
Connections:
- D2 pad 2: Net-(D1-A) (its old number) -> Net-(D2-A)
- J1 pad 3: unconnected-(J1-POW-A) -> /LED_CNTRL
- J1 pad 7: /POW_B -> unconnected-(J1-POW-B)
- J1 pad 8: Net-(D1-A) (its old number) -> Net-(D1-K)
- R1 pad 1: Net-(R2-Pad1) -> Net-(D1-K)
- R1 pad 2: Net-(Q1-B) -> Net-(D2-A)
- U1 pad 1: unconnected-(U1-NULL)_1 -> Net-(U1-LX)
- U1 pad 2: Net-(Q1-E) -> GND
- U1 pad 3: Net-(U1-+) -> /LED_CNTRL
- U1 pad 4: GND -> Net-(D2-A)
- U1 pad 5: unconnected-(U1-NULL) -> Net-(D1-K)
Routing:
- net Net-(D2-A): track 0.00 -> 145.8 mm, vias 0 -> 1
- net Net-(D1-A) (its old number): track 130.1 -> 0.00 mm
- net /LED_CNTRL: track 0.00 -> 36.7 mm, vias 0 -> 1
- net Net-(D1-K): track 0.00 -> 33.2 mm
- net Net-(U1-+): track 24.5 -> 0.00 mm
- net /GRAB: track 48.7 -> 70.1 mm
- net Net-(J1-5V): track 32.1 -> 12.2 mm
- net Net-(Q1-E): track 18.6 -> 0.00 mm
- net /SYNC: track 51.6 -> 67.9 mm, vias 0 -> 2
- net Net-(Q1-B): track 12.3 -> 0.00 mm
- net /POW_B: track 9.60 -> 0.00 mm
- net Net-(U1-LX): track 0.00 -> 9.37 mm
- net Net-(R1-Pad2): track 8.61 -> 0.00 mm
- net Net-(D2-K): track 97.5 -> 100.9 mm
- net Net-(R2-Pad1): track 3.33 -> 0.00 mm
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Other:
- board size 203.8 x 22.2 mm -> 191.1 x 22.2 mm
- board text added: "+"
- board text added: "Camera Link v1.5 Jan 2023"
- board text removed: "Camera Link v1.3"

Commit message: PCB v1.6
Parts:
- added GND2: TestPoint, Connector_Pin:Pin_D1.0mm_L10.0mm, F.Cu at (189.2, 121.9)
- R2: value R_US -> 10KΩ
- moved GND1 10.7 mm to (189.2, 109.2)
- moved GRAB1 6.73 mm to (176.5, 109.2)
- moved SYNC1 3.07 mm to (176.5, 121.9)
Connections:
- net Net-(D1-K) renamed /12VDC
- net Net-(J1-5V) renamed /5VDC
- D4 pad 1: Net-(D1-A) -> Net-(D4-K)
- L1 pad 1: Net-(D1-A) -> Net-(D4-K)
- L1 pad 2: Net-(U1-LX) -> Net-(D1-A)
- U1 pad 1: Net-(U1-LX) -> Net-(D1-A)
Routing:
- net Net-(D4-K): track 0.00 -> 27.2 mm
- net Net-(D1-A): track 38.3 -> 12.8 mm, vias 1 -> 0
- net Net-(U1-LX): track 9.37 -> 0.00 mm
- net Net-(D2-K): track 100.9 -> 104.8 mm
- net /GRAB: track 70.1 -> 71.2 mm
- net /SYNC: track 67.9 -> 67.3 mm
Other:
- board text added: "12V"
- board text added: "5V"
- board text added: "Camera Link v1.6 Jan 2023"
- board text added: "GND"
- board text added: "GRAB"
- board text added: "LED"
- board text added: "POW-B"
- board text added: "SPECIAL"
- board text added: "SYNC"
- board text removed: "Camera Link v1.5 Jan 2023"

Commit message: pcb v1.7
Parts:
- removed D1: D, Diode_SMD:D_SMB
- removed L1: L, Inductor_THT:L_Axial_L14.5mm_D5.8mm_P7.62mm_Vertical_Fastron_HBCC
- removed R2: 10KΩ, Resistor_SMD:R_0805_2012Metric
- removed U1: AL8861, Package_TO_SOT_SMD:SOT-89-5
- R1: value R_US -> 5Ω
- moved R1 9.15 mm to (95.8, 112.7)
- moved J1 1.91 mm to (118.6, 111.1)
- moved D2 0.46 mm to (227.3, 115.8)
- moved D3 0.20 mm to (150.2, 115.8)
- moved D4 0.20 mm to (73.0, 115.8)
- moved H1 0.20 mm to (240.0, 115.8)
- moved H2 0.20 mm to (59.7, 115.8)
- moved J2 0.20 mm to (168.4, 115.8)
Connections:
- J1 pad 3: /LED_CNTRL -> Net-(D4-K)
- J1 pad 6: /5VDC -> unconnected-(J1-5V-Pad6)
- J1 pad 7: unconnected-(J1-POW-B) -> Net-(D4-K)
Routing:
- net Net-(D4-K): track 27.2 -> 66.5 mm
- net /LED_CNTRL: track 36.7 -> 0.00 mm, vias 1 -> 0
- net Net-(D1-A): track 12.8 -> 0.00 mm
- net /5VDC: track 12.2 -> 0.00 mm
- net Net-(D2-K): track 104.8 -> 97.7 mm
- net /GRAB: track 71.2 -> 76.8 mm
- net Net-(D2-A): track 145.6 -> 150.3 mm
- net Net-(D3-K): track 104.2 -> 99.7 mm, vias 0 -> 1
- net /12VDC: track 33.2 -> 29.9 mm
- net /SYNC: track 67.3 -> 67.9 mm, vias 2 -> 0
Other:
- board size 191.1 x 22.2 mm -> 189.2 x 19 mm
- board text added: "Camera Link v1.7 Mar 2023"
- board text added: "POW-A"
- board text removed: "Camera Link v1.6 Jan 2023"
- board text removed: "LED"

Commit message: pcb v1.7
Parts:
- renumbered D2 to D1, D3 to D2, D4 to D3, J2 to J1, J1 to J2
