File: pcb/camera_link.kicad_sch (KiCad schematic)
At the start: 12 parts, among them J1 RJ45_pyControl, J2 Screw_Terminal_01x08

Commit message: pcbv1.2
Parts:
- removed R2: 22Ω, Resistor_THT:R_Axial_DIN0204_L3.6mm_D1.6mm_P7.62mm_Horizontal, symbol Device:R_US
- added D10, D11, D12, D13, D14, D15, D16, D17, D18, D19, D20, D21, D22, D23, D24, D7, D8, D9: LED, LED_SMD:LED_1206_3216Metric, symbol Device:LED
- J1: footprint asl_footprints:RJ45_THP_Vertical -> asl_footprints:RJ45_SMD
- R1: value 22Ω -> 9Ω; footprint Resistor_THT:R_Axial_DIN0204_L3.6mm_D1.6mm_P7.62mm_Horizontal -> Resistor_SMD:R_1206_3216Metric_Pad1.30x1.75mm_HandSolder
Connections:
- net GND: now reaches J1.2 (GND), J2.2 (Pin_2)
- net at J1.7 (POW-B), J2.7 (Pin_7): now also R1.2; no longer R1.1
- net at J1.8 (12V), J2.8 (Pin_8): now also D1.2 (A), D2.2 (A), D3.2 (A), D4.2 (A)
- net at D5.1 (K), D6.1 (K): now also D10.2 (A), D11.2 (A), D12.2 (A), D7.1 (K), D8.1 (K), D9.2 (A); no longer D4.1 (K)
- net at D1.1 (K), D2.1 (K), D3.1 (K): now also D4.1 (K), D5.2 (A), D6.2 (A), D7.2 (A), D8.2 (A); no longer R1.2
- removed net 5VDC: D1.2 (A), D2.2 (A), D3.2 (A), D4.2 (A), D5.2 (A), D6.2 (A), J1.6 (5V), J2.6 (Pin_6)
- new net: D17.1 (K), D18.1 (K), D19.1 (K), D20.1 (K), D21.2 (A), D22.2 (A), D23.2 (A), D24.2 (A)
- new net: D13.1 (K), D14.1 (K), D15.1 (K), D16.1 (K), D17.2 (A), D18.2 (A), D19.2 (A), D20.2 (A)
- new net: D10.1 (K), D11.1 (K), D12.1 (K), D13.2 (A), D14.2 (A), D15.2 (A), D16.2 (A), D9.1 (K)
- new net: J1.6 (5V), J2.6 (Pin_6)
- new net: D21.1 (K), D22.1 (K), D23.1 (K), D24.1 (K), R1.1
Other:
- moved on the sheet: D1, D2, D3, H1, H2, J1, J2, R1

Commit message: pcb v1.3
Parts:
- removed D10, D11, D12, D13, D14, D15, D16, D17, D18, D19, D20, D21, D22, D23, D24, D4, D5, D6, D7, D8, D9: LED, LED_SMD:LED_1206_3216Metric, symbol Device:LED
- removed J2: Screw_Terminal_01x08, Connector_PinHeader_1.27mm:PinHeader_1x08_P1.27mm_Vertical, symbol Connector:Screw_Terminal_01x08
- added GND_TEST1, GRAB1, SYNC1, TP1, TP2: TestPoint, Connector_Pin:Pin_D1.0mm_L10.0mm, symbol Connector:TestPoint
- added J2, J3: Conn_01x09_Female, asl_footprints:JST_NSH_1x09_VERTICAL, symbol Connector:Conn_01x09_Female
- added Q1: 2N2219, Package_TO_SOT_SMD:SOT-23-6, symbol asl_symbols_new:NPN_transistor_ZXTC2045E6TA
- added R2: 100, Resistor_SMD:R_0805_2012Metric, symbol Device:R_US
- added R3: MP915-4.00-1%, asl_footprints:Resistor_power_MP900, symbol Device:R_US
- added RV1: 3386P-1-504TLF, Potentiometer_THT:Potentiometer_Bourns_3386P_Vertical, symbol Device:R_Potentiometer_Trim_US
- added U1: LM741, Package_DIP:DIP-8_W7.62mm, symbol Amplifier_Operational:LM741
- D1, D2, D3: value LED -> LST1-01F09-IR01-00; footprint LED_SMD:LED_1206_3216Metric -> asl_footprints:LED_starboard
- H1: renamed from H2; value Threaded_Standoff -> 24882; Sim_Device (none) -> SPICE; Sim_Params (none) -> type=H model="24882"
- H2: renamed from H1; value Threaded_Standoff -> 24882; Sim_Device (none) -> SPICE; Sim_Params (none) -> type=H model="24882"
- J1: value RJ45_pyControl -> 54602-908LF; footprint asl_footprints:RJ45_SMD -> asl_footprints:RJ45_THP
- R1: value 9Ω -> 5K; footprint Resistor_SMD:R_1206_3216Metric_Pad1.30x1.75mm_HandSolder -> Resistor_SMD:R_0805_2012Metric
Connections:
- net GND: now also GND_TEST1.1, J2.3 (Pin_3), J2.4 (Pin_4), J3.6 (Pin_6), J3.7 (Pin_7), RV1.3, TP2.1, U1.4 (V-)
- net GRAB: now reaches J1.1 (DIO-A)
- net GRAB: now also GRAB1.1, J2.6 (Pin_6), J3.4 (Pin_4)
- net SYNC: now reaches J1.4 (DIO-B)
- net SYNC: now also J2.1 (Pin_1), J3.9 (Pin_9), SYNC1.1
- net at J1.6 (5V): now also R1.1, U1.7 (V+)
- net at R1.2: now also RV1.1; no longer J1.7 (POW-B)
- net at D1.2 (A), J1.8 (12V): no longer D2.2 (A), D3.2 (A)
- new net: D2.1 (K), D3.2 (A)
- new net: D1.1 (K), D2.2 (A)
- new net: D3.1 (K), Q1.3 (C)
- new net: Q1.1 (E), R3.2, U1.2 (-)
- new net: RV1.2, TP1.1, U1.3 (+)
- new net: Q1.2 (B), R2.2
- new net: R2.1, U1.6
- new net POW_B: J1.7 (POW-B), R3.1
Other:
- moved on the sheet: H1, H2

Commit message: pcb v1.5
Parts:
- removed D1: LST1-01F09-IR01-00, asl_footprints:LED_starboard, symbol Device:LED
- removed J3: Conn_01x09_Female, asl_footprints:JST_NSH_1x09_VERTICAL, symbol Connector:Conn_01x09_Female
- removed Q1: 2N2219, Package_TO_SOT_SMD:SOT-23-6, symbol asl_symbols_new:NPN_transistor_ZXTC2045E6TA
- removed R3: MP915-4.00-1%, asl_footprints:Resistor_power_MP900, symbol Device:R_US
- removed RV1: 3386P-1-504TLF, Potentiometer_THT:Potentiometer_Bourns_3386P_Vertical, symbol Device:R_Potentiometer_Trim_US
- removed TP1, TP2: TestPoint, Connector_Pin:Pin_D1.0mm_L10.0mm, symbol Connector:TestPoint
- removed U1: LM741, Package_DIP:DIP-8_W7.62mm, symbol Amplifier_Operational:LM741
- added D1: D, Diode_SMD:D_SMB, symbol Device:D
- added D4: LST1-01F09-IR01-00, asl_footprints:LED_starboard, symbol Device:LED
- added L1: L, Inductor_THT:L_Axial_L14.5mm_D5.8mm_P7.62mm_Vertical_Fastron_HBCC, symbol Device:L
- added U1: AL8861, Package_TO_SOT_SMD:SOT-89-5, symbol asl_symbols_new:AL8861
- H1: renamed from H2; Sim_Device SPICE -> (none); Sim_Params type=H model="24882" -> (none)
- H2: renamed from H1; Sim_Device SPICE -> (none); Sim_Params type=H model="24882" -> (none)
- J1: value 54602-908LF -> E5J88-00LJG2-L; footprint asl_footprints:RJ45_THP -> asl_footprints:RJ45_THP_tab_on_top
- R1: value 5K -> R_US; footprint Resistor_SMD:R_0805_2012Metric -> Resistor_THT:R_Axial_DIN0614_L14.3mm_D5.7mm_P7.62mm_Vertical
- R2: value 100 -> 10KΩ
- renumbered GND_TEST1 to GND1
Connections:
- net GND: now also U1.2 (GND)
- net at D2.2 (A): now also R1.2, U1.4 (Isense)
- net at J1.8 (12V): now also R1.1, D1.1 (K), U1.5 (Vin)
- net at J1.6 (5V): now also R2.1; no longer R1.1
- net at D3.1 (K): now also D4.2 (A)
- net LED_CNTRL: now reaches R2.2
- net LED_CNTRL: now also J1.3 (POW-A), U1.3 (Vset)
- net POW_B: no longer names the net of J1.7 (POW-B)
- new net: L1.2, U1.1 (LX)
- new net: D1.2 (A), D4.1 (K), L1.1
Other:
- moved on the sheet: GND1, GRAB1, H1, H2, J1, J2

Commit message: PCB v1.6
Parts:
- added GND2: TestPoint, Connector_Pin:Pin_D1.0mm_L10.0mm, symbol Connector:TestPoint
Connections:
- net GND: now also GND2.1
- net at L1.2, U1.1 (LX): now also D1.2 (A)
- net 12VDC: now reaches D1.1 (K), J1.8 (12V), R1.1, U1.5 (Vin)
- net at D4.1 (K), L1.1: no longer D1.2 (A)
- net 5VDC: now reaches J1.6 (5V), R2.1
Changed lines of the file:
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@@
   (paper "A5")
   (title_block
-    (date "2023-01-04")
-    (rev "1.5")
-  )
-  (junction (at 57.785 97.79) (diameter 0) (color 0 0 0 0)
+    (date "2023-01-12")
+    (rev "1.6")
+  )
+  (junction (at 56.515 100.33) (diameter 0) (color 0 0 0 0)
+  )
+  (junction (at 56.515 101.6) (diameter 0) (color 0 0 0 0)
+  )
+  (junction (at 132.08 51.435) (diameter 0) (color 0 0 0 0)
   )
   (junction (at 104.775 41.275) (diameter 0) (color 0 0 0 0)
   )
-  (junction (at 53.34 97.79) (diameter 0) (color 0 0 0 0)
-  )
   (junction (at 86.995 38.1) (diameter 0) (color 0 0 0 0)
   )
@@
   (junction (at 86.995 46.355) (diameter 0) (color 0 0 0 0)
   )
-  (junction (at 132.08 41.275) (diameter 0) (color 0 0 0 0)
+  (junction (at 56.515 97.79) (diameter 0) (color 0 0 0 0)
   )
   (wire (pts (xy 86.995 32.385) (xy 86.995 38.1))
@@
     (stroke (width 0) (type default))
   )
+  (wire (pts (xy 56.515 102.235) (xy 56.515 101.6))
+    (stroke (width 0) (type default))
+  )
+  (wire (pts (xy 56.515 101.6) (xy 53.34 101.6))
+    (stroke (width 0) (type default))
+  )
+  (wire (pts (xy 56.515 100.33) (xy 56.515 97.79))
+    (stroke (width 0) (type default))
+  )
   (wire (pts (xy 104.775 51.435) (xy 132.08 51.435))
     (stroke (width 0) (type default))
@@
     (stroke (width 0) (type default))
   )
-  (wire (pts (xy 132.08 41.275) (xy 132.08 32.385))
-    (stroke (width 0) (type default))
-  )
   (wire (pts (xy 132.08 41.275) (xy 132.08 41.91))
     (stroke (width 0) (type default))
   )
-  (wire (pts (xy 57.785 97.79) (xy 69.85 97.79))
-    (stroke (width 0) (type default))
-  )
-  (wire (pts (xy 58.42 105.41) (xy 69.85 105.41))
-    (stroke (width 0) (type default))
-  )
-  (wire (pts (xy 53.34 97.79) (xy 57.785 97.79))
+  (wire (pts (xy 111.125 32.385) (xy 139.065 32.385))
+    (stroke (width 0) (type default))
+  )
+  (wire (pts (xy 64.77 105.41) (xy 69.85 105.41))
+    (stroke (width 0) (type default))
+  )
+  (wire (pts (xy 139.065 51.435) (xy 132.08 51.435))
     (stroke (width 0) (type default))
   )
@@
     (stroke (width 0) (type default))
   )
-  (wire (pts (xy 132.08 32.385) (xy 111.125 32.385))
-    (stroke (width 0) (type default))
-  )
   (wire (pts (xy 53.975 56.515) (xy 59.69 56.515))
     (stroke (width 0) (type default))
@@
     (stroke (width 0) (type default))
   )
+  (wire (pts (xy 139.065 32.385) (xy 139.065 51.435))
+    (stroke (width 0) (type default))
+  )
+  (wire (pts (xy 56.515 97.79) (xy 69.85 97.79))
+    (stroke (width 0) (type default))
+  )
+  (wire (pts (xy 56.515 101.6) (xy 56.515 100.33))
+    (stroke (width 0) (type default))
+  )
   (wire (pts (xy 86.995 38.1) (xy 86.995 46.355))
     (stroke (width 0) (type default))
@@
     (stroke (width 0) (type default))
   )
-  (wire (pts (xy 57.785 97.79) (xy 57.785 100.33))
-    (stroke (width 0) (type default))
-  )
   (wire (pts (xy 53.975 59.055) (xy 86.995 59.055))
     (stroke (width 0) (type default))
@@
     (stroke (width 0) (type default))
   )
-  (wire (pts (xy 57.785 100.33) (xy 69.85 100.33))
+  (wire (pts (xy 56.515 100.33) (xy 69.85 100.33))
     (stroke (width 0) (type default))
   )
@@
     (stroke (width 0) (type default))
   )
+  (wire (pts (xy 56.515 97.79) (xy 53.34 97.79))
+    (stroke (width 0) (type default))
+  )
   (wire (pts (xy 62.23 51.435) (xy 53.975 51.435))
     (stroke (width 0) (type default))
   )
-  (label "SYNC" (at 58.42 105.41 180) (fields_autoplaced)
+  (label "SYNC" (at 64.77 105.41 180) (fields_autoplaced)
     (effects (font (size 1.27 1.27)) (justify right bottom))
   )
@@
   )
   (label "GRAB" (at 56.515 64.135 0) (fields_autoplaced)
+    (effects (font (size 1.27 1.27)) (justify left bottom))
+  )
+  (label "5VDC" (at 55.245 51.435 0) (fields_autoplaced)
+    (effects (font (size 1.27 1.27)) (justify left bottom))
+  )
+  (label "12VDC" (at 55.88 46.355 0) (fields_autoplaced)
     (effects (font (size 1.27 1.27)) (justify left bottom))
   )
@@
       (effects (font (size 1.27 1.27)) hide)
     )
-    (property "Datasheet" "~" (at 96.52 38.1 0)
+    (property "Datasheet" "https://www.digikey.com/en/products/detail/ohmite/13FR100E/822906" (at 96.52 38.1 0)
       (effects (font (size 1.27 1.27)) hide)
     )
@@
     )
   )
+  (symbol (lib_id "Connector:TestPoint") (at 53.34 101.6 90) (unit 1)
+    (in_bom yes) (on_board yes) (dnp no)
+    (property "Reference" "GND2" (at 42.545 99.695 90)
+      (effects (font (size 1.27 1.27)))
+    )
+    (property "Value" "TestPoint" (at 50.038 99.8761 90)
+      (effects (font (size 1.27 1.27)))
+    )
+    (property "Footprint" "Connector_Pin:Pin_D1.0mm_L10.0mm" (at 53.34 96.52 0)
+      (effects (font (size 1.27 1.27)) hide)
+    )
+    (property "Datasheet" "" (at 53.34 96.52 0)
+      (effects (font (size 1.27 1.27)) hide)
+    )
+    (pin "1")
+    (instances
+      (project "camera_link"
+        (path "/99c0100e-3cd8-4e53-82df-0857c6b5e0d5"
+          (reference "GND2") (unit 1)
+        )
+      )
+    )
+  )
   (symbol (lib_id "Device:LED") (at 109.855 41.275 180) (unit 1)
     (in_bom yes) (on_board yes) (dnp no)
@@
   )
   (symbol (lib_id "Connector:TestPoint") (at 55.88 92.71 90) (unit 1)
-    (in_bom yes) (on_board yes) (dnp no) (fields_autoplaced)
-    (property "Reference" "GRAB1" (at 52.578 89.0651 90)
+    (in_bom yes) (on_board yes) (dnp no)
+    (property "Reference" "GRAB1" (at 43.815 90.805 90)
       (effects (font (size 1.27 1.27)))
     )
@@
       (effects (font (size 1.27 1.27)) hide)
     )
-    (property "Datasheet" "~" (at 132.08 45.72 0)
+    (property "Datasheet" "https://www.digikey.com/en/products/detail/abracon-llc/aiap-02-330k/3059871" (at 132.08 45.72 0)
       (effects (font (size 1.27 1.27)) hide)
     )
@@
   )
   (symbol (lib_id "Connector:TestPoint") (at 53.34 97.79 90) (unit 1)
-    (in_bom yes) (on_board yes) (dnp no) (fields_autoplaced)
-    (property "Reference" "GND1" (at 50.038 94.1451 90)
+    (in_bom yes) (on_board yes) (dnp no)
+    (property "Reference" "GND1" (at 42.545 95.885 90)
       (effects (font (size 1.27 1.27)))
     )
@@
     )
   )
-  (symbol (lib_id "power:GND") (at 53.34 97.79 0) (unit 1)
-    (in_bom yes) (on_board yes) (dnp no) (fields_autoplaced)
-    (property "Reference" "#PWR0103" (at 53.34 104.14 0)
-      (effects (font (size 1.27 1.27)) hide)
-    )
-    (property "Value" "GND" (at 53.34 101.8461 0)
-      (effects (font (size 1.27 1.27)))
-    )
-    (property "Footprint" "" (at 53.34 97.79 0)
-      (effects (font (size 1.27 1.27)) hide)
-    )
-    (property "Datasheet" "" (at 53.34 97.79 0)
-      (effects (font (size 1.27 1.27)) hide)
-    )
+  (symbol (lib_id "power:GND") (at 56.515 102.235 0) (unit 1)
+    (in_bom yes) (on_board yes) (dnp no) (fields_autoplaced)
+    (property "Reference" "#PWR0103" (at 56.515 108.585 0)
+      (effects (font (size 1.27 1.27)) hide)
+    )
+    (property "Value" "GND" (at 56.515 106.2911 0)
+      (effects (font (size 1.27 1.27)))
+    )
+    (property "Footprint" "" (at 56.515 102.235 0)
+      (effects (font (size 1.27 1.27)) hide)
+    )
+    (property "Datasheet" "" (at 56.515 102.235 0)
+      (effects (font (size 1.27 1.27)) hide)
+    )

Commit message: pcb v1.7
Parts:
- removed D1: D, Diode_SMD:D_SMB, symbol Device:D
- removed L1: L, Inductor_THT:L_Axial_L14.5mm_D5.8mm_P7.62mm_Vertical_Fastron_HBCC, symbol Device:L
- removed R2: 10KΩ, Resistor_SMD:R_0805_2012Metric, symbol Device:R_US
- removed U1: AL8861, Package_TO_SOT_SMD:SOT-89-5, symbol asl_symbols_new:AL8861
- R1: value R_US -> 5Ω
Connections:
- net LED_CNTRL is gone; now on an unnamed net: J1.3 (POW-A)
- net at D4.1 (K): now also J1.7 (POW-B)
- net 5VDC: no longer names the net of J1.6 (5V)
Other:
- moved on the sheet: D2, D3, D4, GND1, GND2, GRAB1, H1, H2, J2, R1

Commit message: pcb v1.7
Parts:
- GND1, GND2, GRAB1, SYNC1: DNP (none) -> 1
- J1: renamed from J2; value Conn_01x09_Female -> BM09B-NSHSS-TBT
- renumbered D2 to D1, D3 to D2, D4 to D3, J1 to J2
Other:
- note added: "plug"
- note added: "pre-crimped leads"
Changed lines of the file:
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@@
     (stroke (width 0) (type default))
+  )
+  (text "pre-crimped leads" (at 127 88.9 0)
+    (effects (font (size 1.27 1.27)) (justify left bottom) (href "https://www.digikey.com/en/products/detail/jst-sales-america-inc/ASSHLSSHL28K203/9924242?s=N4IgjCBcoOw1oDGUBmBDANgZwKYBoQB7KAbRACYAOcgBgFYBmEAXQIAcAXKEAZQ4CcAlgDsA5iAC+BGJQQhkkdNnxFS4AGwM6MdS3ZdIvASPFSQDMPGjzUmXAWKQyAFhrOds1iE7c+QsZIEALQQ1gpK9qpOIM50dCxmQc5y4XYqjmRg6mD0CRISQA"))
+  )
+  (text "plug" (at 127 86.36 0)
+    (effects (font (size 1.27 1.27)) (justify left bottom) (href "https://www.digikey.com/en/products/detail/jst-sales-america-inc/NSHR-09V-S/3313624"))
   )
   (label "SYNC" (at 140.97 64.77 180) (fields_autoplaced)
@@
       (effects (font (size 1.27 1.27)) hide)
     )
+    (property "Description" "5 watt resistor" (at 67.945 46.355 0)
+      (effects (font (size 1.27 1.27)) hide)
+    )
+    (property "DNP" "" (at 67.945 46.355 0)
+      (effects (font (size 1.27 1.27)) hide)
+    )
     (pin "1")
     (pin "2")
@@
       (effects (font (size 1.27 1.27)) hide)
     )
+    (property "DNP" "1" (at 129.54 60.96 0)
+      (effects (font (size 1.27 1.27)) hide)
+    )
     (pin "1")
     (instances
@@
   (symbol (lib_id "Device:LED") (at 76.835 46.355 180) (unit 1)
     (in_bom yes) (on_board yes) (dnp no)
-    (property "Reference" "D2" (at 78.4225 41.3639 0)
+    (property "Reference" "D1" (at 78.4225 41.3639 0)
       (effects (font (size 1.27 1.27)))
     )
@@
       (effects (font (size 1.27 1.27)) hide)
     )
-    (pin "1")
-    (pin "2")
-    (instances
-      (project "camera_link"
-        (path "/99c0100e-3cd8-4e53-82df-0857c6b5e0d5"
-          (reference "D2") (unit 1)
+    (property "Description" "850 nm LED" (at 76.835 46.355 0)
+      (effects (font (size 1.27 1.27)) hide)
+    )
+    (property "DNP" "" (at 76.835 46.355 0)
+      (effects (font (size 1.27 1.27)) hide)
+    )
+    (pin "1")
+    (pin "2")
+    (instances
+      (project "camera_link"
+        (path "/99c0100e-3cd8-4e53-82df-0857c6b5e0d5"
+          (reference "D1") (unit 1)
         )
       )
@@
       (effects (font (size 1.27 1.27)) hide)
     )
+    (property "DNP" "1" (at 132.08 52.07 0)
+      (effects (font (size 1.27 1.27)) hide)
+    )
     (pin "1")
     (instances
@@
   (symbol (lib_id "Connector:Conn_01x09_Female") (at 151.13 54.61 0) (mirror x) (unit 1)
     (in_bom yes) (on_board yes) (dnp no)
-    (property "Reference" "J2" (at 150.495 41.1607 0)
-      (effects (font (size 1.27 1.27)))
-    )
-    (property "Value" "Conn_01x09_Female" (at 150.495 42.9229 0)
+    (property "Reference" "J1" (at 150.495 41.1607 0)
+      (effects (font (size 1.27 1.27)))
+    )
+    (property "Value" "BM09B-NSHSS-TBT" (at 150.495 42.9229 0)
       (effects (font (size 1.27 1.27)) hide)
     )
@@
     )
     (property "Datasheet" "https://www.digikey.com/en/products/detail/jst-sales-america-inc/BM09B-NSHSS-TBT-LF-SN/3313615" (at 151.13 54.61 0)
+      (effects (font (size 1.27 1.27)) hide)
+    )
+    (property "Description" "9-pin socket" (at 151.13 54.61 0)
+      (effects (font (size 1.27 1.27)) hide)
+    )
+    (property "DNP" "" (at 151.13 54.61 0)
       (effects (font (size 1.27 1.27)) hide)
     )
@@
       (project "camera_link"
         (path "/99c0100e-3cd8-4e53-82df-0857c6b5e0d5"
-          (reference "J2") (unit 1)
+          (reference "J1") (unit 1)
         )
       )
@@
       (effects (font (size 1.27 1.27)) hide)
     )
+    (property "DNP" "1" (at 129.54 57.15 0)
+      (effects (font (size 1.27 1.27)) hide)
+    )
     (pin "1")
     (instances
@@
   (symbol (lib_id "Device:LED") (at 85.725 46.355 180) (unit 1)
     (in_bom yes) (on_board yes) (dnp no)
-    (property "Reference" "D3" (at 87.3125 41.3639 0)
+    (property "Reference" "D2" (at 87.3125 41.3639 0)
       (effects (font (size 1.27 1.27)))
     )
@@
       (effects (font (size 1.27 1.27)) hide)
     )
-    (pin "1")
-    (pin "2")
-    (instances
-      (project "camera_link"
-        (path "/99c0100e-3cd8-4e53-82df-0857c6b5e0d5"
-          (reference "D3") (unit 1)
+    (property "Description" "850 nm LED" (at 85.725 46.355 0)
+      (effects (font (size 1.27 1.27)) hide)
+    )
+    (property "DNP" "" (at 85.725 46.355 0)
+      (effects (font (size 1.27 1.27)) hide)
+    )
+    (pin "1")
+    (pin "2")
+    (instances
+      (project "camera_link"
+        (path "/99c0100e-3cd8-4e53-82df-0857c6b5e0d5"
+          (reference "D2") (unit 1)
         )
       )
@@
       (effects (font (size 1.27 1.27)) hide)
     )
+    (property "DNP" "" (at 81.915 84.455 0)
+      (effects (font (size 1.27 1.27)) hide)
+    )
     (instances
       (project "camera_link"
@@
       (effects (font (size 1.27 1.27)) hide)
     )
+    (property "DNP" "1" (at 140.97 64.77 0)
+      (effects (font (size 1.27 1.27)) hide)
+    )
     (pin "1")
     (instances
@@
     )
     (property "Sim.Params" "type=H model=\"24882\"" (at -29.21 166.37 0)
+      (effects (font (size 1.27 1.27)) hide)
+    )
+    (property "DNP" "" (at 81.915 78.105 0)
       (effects (font (size 1.27 1.27)) hide)
     )
@@
   (symbol (lib_id "power:GND") (at 64.77 61.595 0) (unit 1)
     (in_bom yes) (on_board yes) (dnp no) (fields_autoplaced)
-    (property "Reference" "#PWR0101" (at 64.77 67.945 0)
+    (property "Reference" "#PWR01" (at 64.77 67.945 0)
       (effects (font (size 1.27 1.27)) hide)
     )
@@
       (project "camera_link"
         (path "/99c0100e-3cd8-4e53-82df-0857c6b5e0d5"
-          (reference "#PWR0101") (unit 1)
+          (reference "#PWR01") (unit 1)
         )
       )
@@
   (symbol (lib_id "power:GND") (at 132.715 61.595 0) (unit 1)
     (in_bom yes) (on_board yes) (dnp no) (fields_autoplaced)
-    (property "Reference" "#PWR0103" (at 132.715 67.945 0)
+    (property "Reference" "#PWR02" (at 132.715 67.945 0)
       (effects (font (size 1.27 1.27)) hide)
     )
@@
       (project "camera_link"
         (path "/99c0100e-3cd8-4e53-82df-0857c6b5e0d5"
-          (reference "#PWR0103") (unit 1)
+          (reference "#PWR02") (unit 1)
         )
       )
@@
   (symbol (lib_id "Device:LED") (at 95.25 46.355 180) (unit 1)
     (in_bom yes) (on_board yes) (dnp no)
-    (property "Reference" "D4" (at 96.8375 41.3639 0)
+    (property "Reference" "D3" (at 96.8375 41.3639 0)
       (effects (font (size 1.27 1.27)))
     )
@@
       (effects (font (size 1.27 1.27)) hide)
     )
-    (pin "1")
-    (pin "2")
-    (instances
-      (project "camera_link"
-        (path "/99c0100e-3cd8-4e53-82df-0857c6b5e0d5"
-          (reference "D4") (unit 1)
+    (property "Description" "850 nm LED" (at 95.25 46.355 0)
+      (effects (font (size 1.27 1.27)) hide)
+    )
+    (property "DNP" "" (at 95.25 46.355 0)
+      (effects (font (size 1.27 1.27)) hide)
+    )
+    (pin "1")
+    (pin "2")
+    (instances
+      (project "camera_link"
+        (path "/99c0100e-3cd8-4e53-82df-0857c6b5e0d5"
+          (reference "D3") (unit 1)
         )
       )
@@
   (symbol (lib_name "RJ45_pyControl_1") (lib_id "asl_symbols:RJ45_pyControl") (at 42.545 55.245 0) (unit 1)
     (in_bom yes) (on_board yes) (dnp no) (fields_autoplaced)
-    (property "Reference" "J1" (at 41.91 42.2529 0)
+    (property "Reference" "J2" (at 41.91 42.2529 0)
       (effects (font (size 1.27 1.27)))
     )
@@
     )
     (property "Datasheet" "https://www.digikey.com/en/products/detail/pulse-electronics/E5J88-00LJG2-L/1785312?s=N4IgTCBcDaIKxwMwFoxgGwBZkDkAiIAugL5A" (at 40.005 55.88 90)
+      (effects (font (size 1.27 1.27)) hide)
+    )
+    (property "Description" "RJ45 jack" (at 42.545 55.245 0)
+      (effects (font (size 1.27 1.27)) hide)
+    )
+    (property "DNP" "" (at 42.545 55.245 0)
       (effects (font (size 1.27 1.27)) hide)
     )
@@
       (project "camera_link"
         (path "/99c0100e-3cd8-4e53-82df-0857c6b5e0d5"
-          (reference "J1") (unit 1)
-        )
-      )
+          (reference "J2") (unit 1)
+        )
+      )
